File: hardware/stratospheric_balloon/stratospheric_balloon.sch (KiCad schematic (older format))
At the start: 54 parts, among them J1 Conn_01x04, J2 UFL, J3 SIM_Card, J4 Conn_01x03, J6 Conn_01x02, M1 SIM800C, M2 GY-GPS6MV2, M3 CC1101_MODULE_MIDDLE, M4 MPU6050_MODULE, M5 BME280_MODULE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

Commit message: Add some values
Parts:
- C17, C18, C4: value 22p -> 100n
- R1, R14, R15, R17, R4, R5: value R -> 10k
- R11: value R -> 4.7k
- R12: value R -> 47k
- R13: value R -> 10M
- R16: value R -> 100
- R2, R3: value R -> 1k
- R6, R7, R8: value R -> 51
- R9: value R -> 5.6k
- Y1: value Crystal -> 8MHz
Changed lines of the file:
@@
 U 1 1 5CA6279D
 P 1300 5950
-F 0 "R6" V 1380 5950 50  0000 C CNN
-F 1 "R" V 1300 5950 50  0000 C CNN
+F 0 "R6" V 1050 5850 50  0000 C CNN
+F 1 "51" V 1300 5950 50  0000 C CNN
 F 2 "Resistors_SMD:R_0603" V 1230 5950 50  0001 C CNN
 F 3 "" H 1300 5950 50  0001 C CNN
@@
 U 1 1 5CA627E5
 P 1300 6050
-F 0 "R7" V 1380 6050 50  0000 C CNN
-F 1 "R" V 1300 6050 50  0000 C CNN
+F 0 "R7" V 1000 6050 50  0000 C CNN
+F 1 "51" V 1300 6050 50  0000 C CNN
 F 2 "Resistors_SMD:R_0603" V 1230 6050 50  0001 C CNN
 F 3 "" H 1300 6050 50  0001 C CNN
@@
 U 1 1 5CA62828
 P 1300 6150
-F 0 "R8" V 1380 6150 50  0000 C CNN
-F 1 "R" V 1300 6150 50  0000 C CNN
+F 0 "R8" V 950 6250 50  0000 C CNN
+F 1 "51" V 1300 6150 50  0000 C CNN
 F 2 "Resistors_SMD:R_0603" V 1230 6150 50  0001 C CNN
 F 3 "" H 1300 6150 50  0001 C CNN
@@
 U 1 1 5CA63034
 P 1500 6250
-F 0 "C10" H 1400 6350 50  0000 L CNN
-F 1 "22p" H 1300 6200 50  0000 L CNN
+F 0 "C10" H 1250 6250 50  0000 L CNN
+F 1 "22p" H 1300 6150 50  0000 L CNN
 F 2 "Capacitors_SMD:C_0603" H 1500 6250 50  0001 C CNN
 F 3 "" H 1500 6250 50  0001 C CNN
@@
 U 1 1 5CA63EC3
 P 3850 5950
-F 0 "R12" V 3930 5950 50  0000 C CNN
-F 1 "R" V 3850 5950 50  0000 C CNN
+F 0 "R12" H 4000 5950 50  0000 C CNN
+F 1 "47k" H 4000 6050 50  0000 C CNN
 F 2 "Resistors_SMD:R_0603" V 3780 5950 50  0001 C CNN
 F 3 "" H 3850 5950 50  0001 C CNN
@@
 P 3650 5750
 F 0 "R11" V 3730 5750 50  0000 C CNN
-F 1 "R" V 3650 5750 50  0000 C CNN
+F 1 "4.7k" V 3550 5800 50  0000 C CNN
 F 2 "Resistors_SMD:R_0603" V 3580 5750 50  0001 C CNN
 F 3 "" H 3650 5750 50  0001 C CNN
@@
 U 1 1 5CA68BBF
 P 10250 4000
-F 0 "C17" H 10260 4070 50  0000 L CNN
-F 1 "22p" H 10350 3950 50  0000 L CNN
+F 0 "C17" H 10050 4100 50  0000 L CNN
+F 1 "100n" H 10000 3900 50  0000 L CNN
 F 2 "Capacitors_SMD:C_0603" H 10250 4000 50  0001 C CNN
 F 3 "" H 10250 4000 50  0001 C CNN
@@
 P 10950 4000
 F 0 "C18" H 10960 4070 50  0000 L CNN
-F 1 "22p" H 11050 3950 50  0000 L CNN
+F 1 "100n" H 11000 3900 50  0000 L CNN
 F 2 "Capacitors_SMD:C_0603" H 10950 4000 50  0001 C CNN
 F 3 "" H 10950 4000 50  0001 C CNN
@@
 U 1 1 5CA69B16
 P 10250 3000
-F 0 "R17" V 10330 3000 50  0000 C CNN
-F 1 "R" V 10250 3000 50  0000 C CNN
+F 0 "R17" H 10100 2950 50  0000 C CNN
+F 1 "10k" H 10100 3100 50  0000 C CNN
 F 2 "Resistors_SMD:R_0603" V 10180 3000 50  0001 C CNN
 F 3 "" H 10250 3000 50  0001 C CNN
@@
 P 10050 2800
 F 0 "R16" V 10130 2800 50  0000 C CNN
-F 1 "R" V 10050 2800 50  0000 C CNN
+F 1 "100" V 9950 2800 50  0000 C CNN
 F 2 "Resistors_SMD:R_0603" V 9980 2800 50  0001 C CNN
 F 3 "" H 10050 2800 50  0001 C CNN
@@
 U 1 1 5CA6C0C0
 P 1350 6800
-F 0 "R9" V 1430 6800 50  0000 C CNN
-F 1 "R" V 1350 6800 50  0000 C CNN
+F 0 "R9" H 1500 6750 50  0000 C CNN
+F 1 "5.6k" H 1500 6850 50  0000 C CNN
 F 2 "Resistors_SMD:R_0603" V 1280 6800 50  0001 C CNN
 F 3 "" H 1350 6800 50  0001 C CNN
@@
 U 1 1 5CA6C174
 P 1050 6550
-F 0 "R3" V 1130 6550 50  0000 C CNN
-F 1 "R" V 1050 6550 50  0000 C CNN
+F 0 "R3" V 950 6650 50  0000 C CNN
+F 1 "1k" V 950 6500 50  0000 C CNN
 F 2 "Resistors_SMD:R_0603" V 980 6550 50  0001 C CNN
 F 3 "" H 1050 6550 50  0001 C CNN
@@
 U 1 1 5CA6C67C
 P 1050 6450
-F 0 "R2" V 1130 6450 50  0000 C CNN
-F 1 "R" V 1050 6450 50  0000 C CNN
+F 0 "R2" V 1150 6550 50  0000 C CNN
+F 1 "1k" V 1150 6400 50  0000 C CNN
 F 2 "Resistors_SMD:R_0603" V 980 6450 50  0001 C CNN
 F 3 "" H 1050 6450 50  0001 C CNN
@@
 P 950 3250
 F 0 "R1" V 1030 3250 50  0000 C CNN
-F 1 "R" V 950 3250 50  0000 C CNN
+F 1 "10k" H 850 3400 50  0000 C CNN
 F 2 "Resistors_SMD:R_0603" V 880 3250 50  0001 C CNN
 F 3 "" H 950 3250 50  0001 C CNN
@@
 P 950 4050
 F 0 "C4" H 960 4120 50  0000 L CNN
-F 1 "22p" H 1050 4000 50  0000 L CNN
+F 1 "100n" H 1000 3900 50  0000 L CNN
 F 2 "Capacitors_SMD:C_0603" H 950 4050 50  0001 C CNN
 F 3 "" H 950 4050 50  0001 C CNN
@@
 U 1 1 5CA70366
 P 5800 2950
-F 0 "R15" V 5880 2950 50  0000 C CNN
-F 1 "R" V 5800 2950 50  0000 C CNN
+F 0 "R15" H 5950 3050 50  0000 C CNN
+F 1 "10k" H 5950 2900 50  0000 C CNN
 F 2 "Resistors_SMD:R_0603" V 5730 2950 50  0001 C CNN
 F 3 "" H 5800 2950 50  0001 C CNN
@@
 U 1 1 5CA7116B
 P 1200 3250
-F 0 "R4" H 1280 3250 50  0000 C CNN
-F 1 "R" V 1200 3250 50  0000 C CNN
+F 0 "R4" H 1350 3400 50  0000 C CNN
+F 1 "10k" H 1350 3200 50  0000 C CNN
 F 2 "Resistors_SMD:R_0603" V 1130 3250 50  0001 C CNN
 F 3 "" H 1200 3250 50  0001 C CNN
@@
 U 1 1 5CA71D1A
 P 1200 4050
-F 0 "R5" V 1280 4050 50  0000 C CNN
-F 1 "R" V 1200 4050 50  0000 C CNN
+F 0 "R5" H 1350 4150 50  0000 C CNN
+F 1 "10k" H 1350 4000 50  0000 C CNN
 F 2 "Resistors_SMD:R_0603" V 1130 4050 50  0001 C CNN
 F 3 "" H 1200 4050 50  0001 C CNN
@@
 U 1 1 5CA72659
 P 5800 2550
-F 0 "R14" V 5880 2550 50  0000 C CNN
-F 1 "R" V 5800 2550 50  0000 C CNN
+F 0 "R14" H 5950 2650 50  0000 C CNN
+F 1 "10k" H 5950 2500 50  0000 C CNN
 F 2 "Resistors_SMD:R_0603" V 5730 2550 50  0001 C CNN
 F 3 "" H 5800 2550 50  0001 C CNN
@@
 P 5200 4900
 F 0 "Y1" H 5200 5050 50  0000 C CNN
-F 1 "Crystal" H 5200 4750 50  0000 C CNN
+F 1 "8MHz" H 5200 4750 50  0000 C CNN
 F 2 "Crystals:Crystal_HC49-4H_Vertical" H 5200 4900 50  0001 C CNN
 F 3 "" H 5200 4900 50  0001 C CNN
@@
 U 1 1 5CA732E7
 P 5000 5400
-F 0 "C13" H 5010 5470 50  0000 L CNN
-F 1 "22p" H 5100 5350 50  0000 L CNN
+F 0 "C13" H 4800 5500 50  0000 L CNN
+F 1 "22p" H 4800 5350 50  0000 L CNN
 F 2 "Capacitors_SMD:C_0603" H 5000 5400 50  0001 C CNN
 F 3 "" H 5000 5400 50  0001 C CNN
@@
 P 5400 5400
 F 0 "C14" H 5410 5470 50  0000 L CNN
-F 1 "22p" H 5500 5350 50  0000 L CNN
+F 1 "22p" H 5450 5350 50  0000 L CNN
 F 2 "Capacitors_SMD:C_0603" H 5400 5400 50  0001 C CNN
 F 3 "" H 5400 5400 50  0001 C CNN
@@
 P 5200 5200
 F 0 "R13" V 5280 5200 50  0000 C CNN
-F 1 "R" V 5200 5200 50  0000 C CNN
+F 1 "10M" V 5100 5200 50  0000 C CNN
 F 2 "Resistors_SMD:R_0603" V 5130 5200 50  0001 C CNN
 F 3 "" H 5200 5200 50  0001 C CNN
